File: hardware/board/harp.breakout.mini-clamp/harp.breakout.mini-clamp.kicad_pcb (KiCad board)
At the start: 2 copper layers, 40 x 75 mm, 17 parts, among them J1 Conn_01x12_Socket, J5 Conn_02x10_Odd_Even, J6 Conn_01x12_Socket, U5 TXB0108

Commit message: update mini clamp board
Parts:
- removed U5: TXB0108, Package_SO:TSSOP-20_4.4x6.5mm_P0.65mm
- added C12: 100nF, Capacitor_SMD:C_0402_1005Metric, B.Cu at (131.6, 57.3)
- added C13: 100nF, Capacitor_SMD:C_0402_1005Metric, B.Cu at (127.8, 63.8)
- added C16: 100nF, Capacitor_SMD:C_0402_1005Metric, B.Cu at (131.6, 63.8)
- added C17: 100nF, Capacitor_SMD:C_0402_1005Metric, B.Cu at (127.8, 70.3)
- added C20: 100nF, Capacitor_SMD:C_0402_1005Metric, B.Cu at (131.6, 70.3)
- added C6: 100nF, Capacitor_SMD:C_0402_1005Metric, B.Cu at (127.8, 50.8)
- added C7: 15nF, Capacitor_SMD:C_0402_1005Metric, B.Cu at (134.4, 76.0)
- added C8: 10uF, Capacitor_SMD:C_0805_2012Metric, B.Cu at (151.0, 48.5)
- added C9: 100nF, Capacitor_SMD:C_0402_1005Metric, B.Cu at (131.6, 50.8)
- added D1: D_Zener, Diode_SMD:D_SOD-323, B.Cu at (133.9, 97.0)
- added D2: D_Zener, Diode_SMD:D_SOD-323, B.Cu at (133.9, 90.5)
- added D3: D_Zener, Diode_SMD:D_SOD-323, B.Cu at (133.9, 84.0)
- added D4: D_Zener, Diode_SMD:D_SOD-323, B.Cu at (133.9, 77.5)
- added R10: 10K, Resistor_SMD:R_0402_1005Metric, B.Cu at (136.1, 96.5)
- added R11: 10K, Resistor_SMD:R_0402_1005Metric, B.Cu at (136.1, 83.5)
- added R12: 10K, Resistor_SMD:R_0402_1005Metric, B.Cu at (136.1, 77.0)
- added R2: 50, Resistor_SMD:R_1206_3216Metric, B.Cu at (134.4, 68.5)
- added R5: 50, Resistor_SMD:R_1206_3216Metric, B.Cu at (134.4, 55.5)
- added R7: 50, Resistor_SMD:R_1206_3216Metric, B.Cu at (134.4, 49.0)
- added R9: 10K, Resistor_SMD:R_0402_1005Metric, B.Cu at (136.1, 90.0)
- added U1: 74LVCH2T45DC, Package_SO:VSSOP-8_2.3x2mm_P0.5mm, B.Cu at (129.7, 68.5)
- added U2: 74LVCH2T45DC, Package_SO:VSSOP-8_2.3x2mm_P0.5mm, B.Cu at (129.7, 62.0)
- added U3: 74LVCH2T45DC, Package_SO:VSSOP-8_2.3x2mm_P0.5mm, B.Cu at (129.7, 55.5)
- added U4: 74LVCH2T45DC, Package_SO:VSSOP-8_2.3x2mm_P0.5mm, B.Cu at (129.7, 49.0)
- C1: value 1uF -> 10uF; footprint Capacitor_SMD:C_0402_1005Metric_Pad0.74x0.62mm_HandSolder -> Capacitor_SMD:C_0805_2012Metric
- C2, C3: value 100nF -> 15nF; footprint Capacitor_SMD:C_0402_1005Metric_Pad0.74x0.62mm_HandSolder -> Capacitor_SMD:C_0402_1005Metric
- C4: value 1uF -> 15nF; footprint Capacitor_SMD:C_0402_1005Metric_Pad0.74x0.62mm_HandSolder -> Capacitor_SMD:C_0402_1005Metric
- C5: value 1uF -> 100nF; footprint Capacitor_SMD:C_0402_1005Metric_Pad0.74x0.62mm_HandSolder -> Capacitor_SMD:C_0402_1005Metric
- R1: value 10K -> 50; footprint Resistor_SMD:R_0402_1005Metric_Pad0.72x0.64mm_HandSolder -> Resistor_SMD:R_1206_3216Metric
- moved C5 32.0 mm to (127.8, 57.3)
- moved C3 26.8 mm to (134.5, 89.0)
- moved C2 25.5 mm to (134.5, 95.5), turned to 180 degrees
- moved C1 24.4 mm to (148.9, 48.5)
- moved C4 23.6 mm to (134.5, 82.5), turned to 180 degrees
- moved R1 23.4 mm to (134.4, 62.0)
Connections:
- C2 pad 1: GND -> /IN0
- C2 pad 2: +5V -> GND
- C3 pad 1: GND -> /IN1
- C3 pad 2: +3.3V -> GND
- C4 pad 1: +3.3V -> /IN2
- C5 pad 1: Net-(U5-OE) -> GND
- C5 pad 2: GND -> +3.3V
- R1 pad 1: Net-(U5-OE) -> Net-(U2-1B)
- R1 pad 2: +3.3V -> /OUT1_5V
Routing:
- net +3.3V: track 34.6 -> 133.8 mm
- net /IN0_5V: track 26.2 -> 1.90 mm
- net /OUT3_5V: track 26.2 -> 2.14 mm
- net /IN1_5V: track 20.4 -> 1.90 mm
- net /OUT2_5V: track 20.1 -> 2.14 mm
- net /IN0: track 49.5 -> 65.5 mm
- net /IN1: track 46.4 -> 60.5 mm
- net /IN2_5V: track 14.9 -> 1.90 mm
- net /OUT1_5V: track 14.7 -> 2.14 mm
- net +5V: track 0.00 -> 11.9 mm, vias 2 -> 4
- net /IN2: track 43.8 -> 55.6 mm
- net /IN3: track 41.8 -> 53.3 mm
- net /IN3_5V: track 11.2 -> 1.90 mm
- net /OUT0_5V: track 11.0 -> 2.14 mm
- net /OUT3: track 30.0 -> 24.1 mm
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- added copper zone on B.Cu, net +3.3V
- removed copper zone on B.Cu, net +5V
Other:
- board text added: "0368-E-002-001.001.000"
- board text added: "CAM0"
- board text added: "CAM1"
- board text added: "CAM2"
- board text added: "CAM3"
- board text added: "GPI22"
- board text added: "GPI23"
- board text added: "GPI24"
- board text added: "GPI25"
- board text added: "GPO26"
- board text added: "GPO27"
- board text added: "GPO28"
- board text added: "GPO29"
- board text added: "PIN"
- board text added: "POKE0"
- board text added: "POKE1"
- board text added: "POKE2"
- board text added: "POKE3"
- board text added: "Sonya Vasquez Sept 15, 2025"
- board text added: "· 5V logic poke-input and camera-trigger-output. · compatible connectors: 3M Mini Clamp Socket Series. · 37103-2165-000 FL 100 · 37103-3101-000 FL 100"
- board text removed: "0368-E-002-001.000.000"
- board text removed: "GPIO"
- board text removed: "Sonya Vasquez Mar 3, 2025"
- board text removed: "· 5V logic input/output. · connected devices using pullups must use pullups >50KOhm. · compatible connectors: 3M Mini Clamp Socket Series. · 37103-2165-000 FL 100 · 37103-3101-000 FL 100"
