File: hardware/board/harp.breakout.mini-clamp/harp.breakout.mini-clamp.kicad_sch (KiCad schematic)
At the start: 10 parts, among them J1 Conn_01x12_Socket, J5 Conn_02x10_Odd_Even, J6 Conn_01x12_Socket, U5 TXB0108

Commit message: update mini clamp board
Parts:
- removed U5: TXB0108, Package_SO:TSSOP-20_4.4x6.5mm_P0.65mm, symbol Logic_LevelTranslator:TXB0108DQSR
- added C12, C13, C16, C17, C20, C6, C9: 100nF, Capacitor_SMD:C_0402_1005Metric, symbol Device:C
- added C7: 15nF, Capacitor_SMD:C_0402_1005Metric, symbol Device:C
- added C8: 10uF, Capacitor_SMD:C_0805_2012Metric, symbol Device:C
- added D1, D2, D3, D4: D_Zener, Diode_SMD:D_SOD-323, symbol Device:D_Zener
- added R10, R11, R12, R9: 10K, Resistor_SMD:R_0402_1005Metric, symbol Device:R
- added R2, R5, R7: 50, Resistor_SMD:R_1206_3216Metric, symbol Device:R
- added U1, U2, U3, U4: 74LVCH2T45DC, Package_SO:VSSOP-8_2.3x2mm_P0.5mm, symbol Logic_LevelTranslator:74LVCH2T45DC
- C1: value 1uF -> 10uF; footprint Capacitor_SMD:C_0402_1005Metric_Pad0.74x0.62mm_HandSolder -> Capacitor_SMD:C_0805_2012Metric; Link https://www.digikey.com/en/products/detail/murata-electronics/GRM155R6YA105KE11J/4905163 -> https://www.digikey.com/en/products/detail/murata-electronics/GRM21BZ71E106KE15L/13904911; Manufacturer Number GRM155R6YA105KE11J -> GRM21BZ71E106KE15L; Notes must not be polarized -> (none); Rated Voltage 35V -> 25V; Temperature Coefficient X5R -> X7R
- C2, C3: value 100nF -> 15nF; footprint Capacitor_SMD:C_0402_1005Metric_Pad0.74x0.62mm_HandSolder -> Capacitor_SMD:C_0402_1005Metric; Link https://www.digikey.com/en/products/detail/murata-electroni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 -> (none); Manufacturer Murata Electronics -> Yageo; Manufacturer Number GRM155R71H104KE14D -> CC0402JRX7R7BB153; PCBWay Link https://www.pcbway.com/components/detail/0402B104K160CT/307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 -> (none); Rated Voltage 50V -> (none); Temperature Coefficient X7R -> (none); Tolerance 10% -> (none)
- C4: value 1uF -> 15nF; footprint Capacitor_SMD:C_0402_1005Metric_Pad0.74x0.62mm_HandSolder -> Capacitor_SMD:C_0402_1005Metric; Link https://www.digikey.com/en/products/detail/murata-electroni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 -> (none); Manufacturer Murata Electronics -> Yageo; Manufacturer Number GRM155R6YA105KE11J -> CC0402JRX7R7BB153; Notes must not be polarized -> (none); Rated Voltage 35V -> (none); Temperature Coefficient X5R -> (none)
- C5: value 1uF -> 100nF; footprint Capacitor_SMD:C_0402_1005Metric_Pad0.74x0.62mm_HandSolder -> Capacitor_SMD:C_0402_1005Metric; Link https://www.digikey.com/en/products/detail/murata-electroni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 -> https://www.digikey.com/en/products/detail/walsin-technolog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; Manufacturer Murata Electronics -> Walson Technology Corporation; Manufacturer Number GRM155R6YA105KE11J -> 0402B104K160CT; Notes must not be polarized -> (none); PCBWay Link (none) -> https://www.pcbway.com/components/detail/0402B104K160CT/307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; Rated Voltage 35V -> 16V; Temperature Coefficient X5R -> X7R; Tolerance (none) -> 10%
- R1: value 10K -> 50; footprint Resistor_SMD:R_0402_1005Metric_Pad0.72x0.64mm_HandSolder -> Resistor_SMD:R_1206_3216Metric; Alternate (none) -> HRG3216P-49R9-B-T1; Link https://www.digikey.com/en/products/detail/koa-speer-electr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 -> https://www.digikey.com/en/products/detail/vishay-dale/TNPW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; Manufacturer KOA Speer Electronics, Inc. -> Vishay Dale; Manufacturer Number SG73P1EWTTP1002F -> TNPW120650R0BEEN; Notes (none) -> 1/4W; Tolerance (none) -> 1%
Connections:
- net +3.3V: now also C5.2, C13.2, C17.2, C6.2, C8.1, U1.1 (VCCA), U1.5 (DIR), U2.1 (VCCA), U2.5 (DIR), U3.1 (VCCA), U3.5 (DIR), U4.1 (VCCA), U4.5 (DIR); no longer C3.2, C4.1, R1.2
- net +5V: now also C12.2, C16.2, C20.2, C9.2, U1.8 (VCCB), U2.8 (VCCB), U3.8 (VCCB), U4.8 (VCCB); no longer C2.2
- net GND: now also C2.2, C3.2, C5.1, C12.1, C13.1, C16.1, C17.1, C20.1, C6.1, C7.2, C8.2, C9.1, D1.2 (A), D2.2 (A), D3.2 (A), D4.2 (A), U1.4 (GND), U2.4 (GND), U3.4 (GND), U4.4 (GND); no longer C2.1, C3.1, C5.2
- net IN0: now also C2.1, D1.1 (K), R10.2
- net IN0_5V: now also R10.1
- net IN1: now also C3.1, D2.1 (K), R9.2
- net IN1_5V: now also R9.1
- net IN2: now also C4.1, D3.1 (K), R11.2
- net IN2_5V: now also R11.1
- net IN3: now also C7.1, D4.1 (K), R12.2
- net IN3_5V: now also R12.1
- net OUT0: now also U1.2 (1A), U1.3 (2A)
- net OUT0_5V: now also R2.2
- net OUT1: now also U2.2 (1A), U2.3 (2A)
- net OUT1_5V: now also R1.2
- net OUT2: now also U3.2 (1A), U3.3 (2A)
- net OUT2_5V: now also R5.2
- net OUT3: now also U4.2 (1A), U4.3 (2A)
- net OUT3_5V: now also R7.2
- net at R1.1: now also U2.6 (2B), U2.7 (1B); no longer C5.1
- new net: R2.1, U1.6 (2B), U1.7 (1B)
- new net: R7.1, U4.6 (2B), U4.7 (1B)
- new net: R5.1, U3.6 (2B), U3.7 (1B)
Other:
- note added: "16nF total"
- note added: "V_{z} = 3.3V"
- note removed: "Low pass filter to assert OE after VCC_{A} is stable."
- note removed: "TXBO108DQSR is a 5-V-tolerant (Port B only) bidirectional logic level converter with direction sensing."
- moved on the sheet: J1, J5, J6

Commit message: update breakout
Parts:
- U1, U2, U3, U4: Alternate (none) -> SN74AVC2T45DCUR or SN74LVC2T45DCURG4
Changed lines of the file:
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@@
+			)
+		)
+		(property "Alternate" "SN74AVC2T45DCUR or SN74LVC2T45DCURG4"
+			(at 107.95 35.56 0)
+			(effects
+				(font
+					(size 1.27 1.27)
+				)
+				(hide yes)
 			)
 		)
@@
 			)
 		)
+		(property "Alternate" "SN74AVC2T45DCUR or SN74LVC2T45DCURG4"
+			(at 107.95 77.47 0)
+			(effects
+				(font
+					(size 1.27 1.27)
+				)
+				(hide yes)
+			)
+		)
 		(pin "1"
 		)
@@
 			)
 		)
+		(property "Alternate" "SN74AVC2T45DCUR or SN74LVC2T45DCURG4"
+			(at 107.95 163.83 0)
+			(effects
+				(font
+					(size 1.27 1.27)
+				)
+				(hide yes)
+			)
+		)
 		(pin "1"
 		)
@@
 			(at 107.95 121.92 0)
 			(effects
+				(font
+					(size 1.27 1.27)
+				)
+				(hide yes)
+			)
+		)
+		(property "Alternate" "SN74AVC2T45DCUR or SN74LVC2T45DCURG4"
+			(at 107.95 121.92 0)
+			(effects
